Commit message: new package lab3

File: anro3/urdf/static.urdf (robot description, URDF)
Before this commit: robot robot, 4 links, 3 joints
Joints:
- joint base_to_link1: limit lower=-3.1415 upper=3.1415 effort=1000.0 velocity=0.5 -> (none); type revolute -> fixed
- joint link1_to_link2: limit lower=-1.57075 upper=1.57075 effort=1000.0 velocity=0.5 -> (none); type revolute -> fixed
- joint link2_to_link3: limit lower=0.1 upper=0.2 effort=1000.0 velocity=0.5 -> (none); type prismatic -> fixed
