Commit message: nonkdl working

File: anro3/urdf/moving.urdf (robot description, URDF)
Before this commit: robot robot, 4 links, 3 joints
Joints:
- joint link2_to_link3: limit lower=0.1 upper=0.2 effort=1000.0 velocity=0.5 -> lower=0.06 upper=0.2 effort=1000.0 velocity=0.5

Commit message: nonkdl working

File: anro3/urdf/moving.urdf (robot description, URDF)
Before this commit: robot robot, 4 links, 3 joints
Joints:
- joint link2_to_link3: limit lower=0.06 upper=0.2 effort=1000.0 velocity=0.5 -> lower=0.05 upper=0.2 effort=1000.0 velocity=0.5
